File: desklamp.sch (KiCad schematic (older format))
At the start: 6 parts, among them J1 Power, J2 Neopixel, J3 SPI_header, U1 ATtiny84A-PU

Commit message: Ditch the ATtiny, go with itsy-bitsy
Parts:
- removed J3: SPI_header, Connector_PinHeader_2.54mm:PinHeader_2x03_P2.54mm_Vertical, symbol custom-symbols:SPI_header
- removed U1: ATtiny84A-PU, Package_DIP:DIP-14_W7.62mm, symbol MCU_Microchip_ATtiny:ATtiny84A-PU
- added RV0, RV1, RV2, RV3: R_POT, TerminalBlock:TerminalBlock_bornier-3_P5.08mm, symbol Device:R_POT
- added U1: itsy_bitsy, Socket:itsy_bitsy, symbol custom-symbols:itsy_bitsy
Connections:
- wire segments 21 -> 40
Changed lines of the file:
@@
-$EndComp
-$Comp
-L MCU_Microchip_ATtiny:ATtiny84A-PU U1
-U 1 1 602F160D
-P 5650 2000
-F 0 "U1" H 5120 2046 50  0000 R CNN
-F 1 "ATtiny84A-PU" H 5120 1955 50  0000 R CNN
-F 2 "Package_DIP:DIP-14_W7.62mm" H 5650 2000 50  0001 C CIN
-F 3 "http://ww1.microchip.com/downloads/en/DeviceDoc/doc8183.pdf" H 5650 2000 50  0001 C CNN
-	1    5650 2000
-	1    0    0    -1
 $EndComp
 $Comp
@@
 	3150 2200 3150 2300
 Connection ~ 3150 2200
-$Comp
-L power:GND #PWR0103
-U 1 1 602F1C7F
-P 5650 3000
-F 0 "#PWR0103" H 5650 2750 50  0001 C CNN
-F 1 "GND" H 5655 2827 50  0000 C CNN
-F 2 "" H 5650 3000 50  0001 C CNN
-F 3 "" H 5650 3000 50  0001 C CNN
-	1    5650 3000
-	1    0    0    -1
-$EndComp
-Wire Wire Line
-	5650 2900 5650 3000
-$Comp
-L power:+5V #PWR0104
-U 1 1 602F1CF4
-P 5650 1100
-F 0 "#PWR0104" H 5650 950 50  0001 C CNN
-F 1 "+5V" H 5665 1273 50  0000 C CNN
-F 2 "" H 5650 1100 50  0001 C CNN
-F 3 "" H 5650 1100 50  0001 C CNN
-	1    5650 1100
-	1    0    0    -1
-$EndComp
 $Comp
 L power:+5V #PWR0105
@@
 Wire Wire Line
 	5550 5100 5900 5100
+Text GLabel 6950 2050 2    50   Input ~ 0
+Signal
+Wire Wire Line
+	5250 5100 5000 5100
+$Comp
+L power:GND #PWR0103
+U 1 1 602F604A
+P 5850 1450
+F 0 "#PWR0103" H 5850 1200 50  0001 C CNN
+F 1 "GND" V 5855 1322 50  0000 R CNN
+F 2 "" H 5850 1450 50  0001 C CNN
+F 3 "" H 5850 1450 50  0001 C CNN
+	1    5850 1450
+	0    1    1    0
+$EndComp
+$Comp
+L custom-symbols:itsy_bitsy U1
+U 1 1 602F6D1C
+P 5950 1050
+F 0 "U1" H 6400 1215 50  0000 C CNN
+F 1 "itsy_bitsy" H 6400 1124 50  0000 C CNN
+F 2 "Socket:itsy_bitsy" H 6150 400 50  0001 C CNN
+F 3 "" H 6150 400 50  0001 C CNN
+	1    5950 1050
+	1    0    0    -1
+$EndComp
+$Comp
+L power:+5V #PWR0104
+U 1 1 602F7258
+P 5850 1250
+F 0 "#PWR0104" H 5850 1100 50  0001 C CNN
+F 1 "+5V" V 5865 1378 50  0000 L CNN
+F 2 "" H 5850 1250 50  0001 C CNN
+F 3 "" H 5850 1250 50  0001 C CNN
+	1    5850 1250
+	0    -1   -1   0
+$EndComp
 Text GLabel 5000 5100 0    50   Input ~ 0
 Signal
-Wire Wire Line
-	5250 5100 5000 5100
-$Comp
-L custom-symbols:SPI_header J3
-U 1 1 602F3289
-P 7400 1800
-F 0 "J3" H 7700 1965 50  0000 C CNN
-F 1 "SPI_header" H 7700 1874 50  0000 C CNN
-F 2 "Connector_PinHeader_2.54mm:PinHeader_2x03_P2.54mm_Vertical" H 7550 1600 50  0001 C CNN
-F 3 "" H 7550 1600 50  0001 C CNN
-	1    7400 1800
-	1    0    0    -1
-$EndComp
-$Comp
-L power:GND #PWR0107
-U 1 1 602F3BA9
-P 8100 2100
-F 0 "#PWR0107" H 8100 1850 50  0001 C CNN
-F 1 "GND" V 8105 1972 50  0000 R CNN
-F 2 "" H 8100 2100 50  0001 C CNN
-F 3 "" H 8100 2100 50  0001 C CNN
-	1    8100 2100
-	0    -1   -1   0
-$EndComp
-$Comp
-L power:+5V #PWR0108
-U 1 1 602F3C36
-P 8100 1900
-F 0 "#PWR0108" H 8100 1750 50  0001 C CNN
-F 1 "+5V" V 8115 2028 50  0000 L CNN
-F 2 "" H 8100 1900 50  0001 C CNN
-F 3 "" H 8100 1900 50  0001 C CNN
-	1    8100 1900
-	0    1    1    0
-$EndComp
-Wire Wire Line
-	6250 1900 7300 1900
-Wire Wire Line
-	6250 2000 6500 2000
-Wire Wire Line
-	6500 2000 6500 2250
-Wire Wire Line
-	6500 2250 8450 2250
-Wire Wire Line
-	8450 2250 8450 2000
-Wire Wire Line
-	8450 2000 8100 2000
-Wire Wire Line
-	6250 1800 7150 1800
-Wire Wire Line
-	7150 1800 7150 2000
-Wire Wire Line
-	7150 2000 7300 2000
-Wire Wire Line
-	6250 2600 7150 2600
-Wire Wire Line
-	7150 2600 7150 2100
-Wire Wire Line
-	7150 2100 7300 2100
+$Comp
+L Device:R_POT RV3
+U 1 1 602F751B
+P 4950 2450
+F 0 "RV3" H 4880 2496 50  0000 R CNN
+F 1 "R_POT" H 4880 2405 50  0000 R CNN
+F 2 "TerminalBlock:TerminalBlock_bornier-3_P5.08mm" H 4950 2450 50  0001 C CNN
+F 3 "~" H 4950 2450 50  0001 C CNN
+	1    4950 2450
+	1    0    0    -1
+$EndComp
+$Comp
+L Device:R_POT RV2
+U 1 1 602F75E6
+P 4950 2000
+F 0 "RV2" H 4880 2046 50  0000 R CNN
+F 1 "R_POT" H 4880 1955 50  0000 R CNN
+F 2 "TerminalBlock:TerminalBlock_bornier-3_P5.08mm" H 4950 2000 50  0001 C CNN
+F 3 "~" H 4950 2000 50  0001 C CNN
+	1    4950 2000
+	1    0    0    -1
+$EndComp
+$Comp
+L Device:R_POT RV1
+U 1 1 602F762E
+P 4950 1550
+F 0 "RV1" H 4880 1596 50  0000 R CNN
+F 1 "R_POT" H 4880 1505 50  0000 R CNN
+F 2 "TerminalBlock:TerminalBlock_bornier-3_P5.08mm" H 4950 1550 50  0001 C CNN
+F 3 "~" H 4950 1550 50  0001 C CNN
+	1    4950 1550
+	1    0    0    -1
+$EndComp
+$Comp
+L Device:R_POT RV0
+U 1 1 602F767B
+P 4950 1100
+F 0 "RV0" H 4880 1146 50  0000 R CNN
+F 1 "R_POT" H 4880 1055 50  0000 R CNN
+F 2 "TerminalBlock:TerminalBlock_bornier-3_P5.08mm" H 4950 1100 50  0001 C CNN
+F 3 "~" H 4950 1100 50  0001 C CNN
+	1    4950 1100
+	1    0    0    -1
+$EndComp
+Wire Wire Line
+	4950 1250 5450 1250
+Wire Wire Line
+	5450 1250 5450 1550
+Wire Wire Line
+	5450 1550 5850 1550
+Wire Wire Line
+	4950 2150 5450 2150
+Wire Wire Line
+	5450 2150 5450 1750
+Wire Wire Line
+	5450 1750 5850 1750
+Wire Wire Line
+	4950 1700 5350 1700
+Wire Wire Line
+	5350 1700 5350 1650
+Wire Wire Line
+	5350 1650 5850 1650
+Wire Wire Line
+	4950 2600 5550 2600
+Wire Wire Line
+	5550 2600 5550 1850
+Wire Wire Line
+	5550 1850 5850 1850
+$Comp
+L power:GND #PWR0109
+U 1 1 602F8A7C
+P 4400 2700
+F 0 "#PWR0109" H 4400 2450 50  0001 C CNN
+F 1 "GND" H 4405 2527 50  0000 C CNN
+F 2 "" H 4400 2700 50  0001 C CNN
+F 3 "" H 4400 2700 50  0001 C CNN
+	1    4400 2700
+	1    0    0    -1
+$EndComp
+$Comp
+L power:+5V #PWR0110
+U 1 1 602FA212
+P 5250 2700
+F 0 "#PWR0110" H 5250 2550 50  0001 C CNN
+F 1 "+5V" H 5265 2873 50  0000 C CNN
+F 2 "" H 5250 2700 50  0001 C CNN
+F 3 "" H 5250 2700 50  0001 C CNN
+	1    5250 2700
+	-1   0    0    1
+$EndComp
+Wire Wire Line
+	5100 1100 5250 1100
+Wire Wire Line
+	5250 1100 5250 1550
+Wire Wire Line
+	5100 1550 5250 1550
+Connection ~ 5250 1550
+Wire Wire Line
+	5250 1550 5250 2000
+Wire Wire Line
+	5100 2000 5250 2000
+Connection ~ 5250 2000
+Wire Wire Line
+	5250 2000 5250 2450
+Wire Wire Line
+	5100 2450 5250 2450
+Connection ~ 5250 2450
+Wire Wire Line
+	5250 2450 5250 2700
+Wire Wire Line
+	4400 900  4950 900
+Wire Wire Line
+	4950 900  4950 950
+Wire Wire Line
+	4400 900  4400 1350
+Wire Wire Line
+	4950 1400 4950 1350
+Wire Wire Line
+	4950 1350 4400 1350
+Connection ~ 4400 1350
+Wire Wire Line
+	4400 1350 4400 1800
+Wire Wire Line
+	4950 1850 4950 1800
+Wire Wire Line
+	4950 1800 4400 1800
+Connection ~ 4400 1800
+Wire Wire Line
+	4400 1800 4400 2250
+Wire Wire Line
+	4950 2300 4950 2250
+Wire Wire Line
+	4950 2250 4400 2250
+Connection ~ 4400 2250
+Wire Wire Line
+	4400 2250 4400 2700
 $EndSCHEMATC

Commit message: Work on pcb and generate gerbers
Parts:
- RV0: value R_POT -> POT0
- RV1: value R_POT -> POT1
- RV2: value R_POT -> POT2
- RV3: value R_POT -> POT3
- U1: symbol custom-symbols:itsy_bitsy -> desklamp-rescue:itsy_bitsy-custom-symbols
Changed lines of the file:
@@
 EESchema Schematic File Version 4
-EELAYER 26 0
+EELAYER 30 0
 EELAYER END
 $Descr A4 11693 8268
@@
 $EndComp
 $Comp
-L custom-symbols:itsy_bitsy U1
-U 1 1 602F6D1C
-P 5950 1050
-F 0 "U1" H 6400 1215 50  0000 C CNN
-F 1 "itsy_bitsy" H 6400 1124 50  0000 C CNN
-F 2 "Socket:itsy_bitsy" H 6150 400 50  0001 C CNN
-F 3 "" H 6150 400 50  0001 C CNN
-	1    5950 1050
-	1    0    0    -1
-$EndComp
-$Comp
 L power:+5V #PWR0104
 U 1 1 602F7258
@@
 P 4950 2450
 F 0 "RV3" H 4880 2496 50  0000 R CNN
-F 1 "R_POT" H 4880 2405 50  0000 R CNN
+F 1 "POT3" H 4880 2405 50  0000 R CNN
 F 2 "TerminalBlock:TerminalBlock_bornier-3_P5.08mm" H 4950 2450 50  0001 C CNN
 F 3 "~" H 4950 2450 50  0001 C CNN
@@
 P 4950 2000
 F 0 "RV2" H 4880 2046 50  0000 R CNN
-F 1 "R_POT" H 4880 1955 50  0000 R CNN
+F 1 "POT2" H 4880 1955 50  0000 R CNN
 F 2 "TerminalBlock:TerminalBlock_bornier-3_P5.08mm" H 4950 2000 50  0001 C CNN
 F 3 "~" H 4950 2000 50  0001 C CNN
@@
 P 4950 1550
 F 0 "RV1" H 4880 1596 50  0000 R CNN
-F 1 "R_POT" H 4880 1505 50  0000 R CNN
+F 1 "POT1" H 4880 1505 50  0000 R CNN
 F 2 "TerminalBlock:TerminalBlock_bornier-3_P5.08mm" H 4950 1550 50  0001 C CNN
 F 3 "~" H 4950 1550 50  0001 C CNN
@@
 P 4950 1100
 F 0 "RV0" H 4880 1146 50  0000 R CNN
-F 1 "R_POT" H 4880 1055 50  0000 R CNN
+F 1 "POT0" H 4880 1055 50  0000 R CNN
 F 2 "TerminalBlock:TerminalBlock_bornier-3_P5.08mm" H 4950 1100 50  0001 C CNN
 F 3 "~" H 4950 1100 50  0001 C CNN
@@
 Wire Wire Line
 	4400 2250 4400 2700
+$Comp
+L desklamp-rescue:itsy_bitsy-custom-symbols U1
+U 1 1 602F6D1C
+P 5950 1050
+F 0 "U1" H 6400 1215 50  0000 C CNN
+F 1 "itsy_bitsy" H 6400 1124 50  0000 C CNN
+F 2 "Socket:itsy_bitsy" H 6150 400 50  0001 C CNN
+F 3 "" H 6150 400 50  0001 C CNN
+	1    5950 1050
+	1    0    0    -1
+$EndComp
 $EndSCHEMATC

Commit message: Added a jumper for POT3 so that it can be used as a second NeoPixel port
Parts:
- removed RV3: POT3, TerminalBlock:TerminalBlock_bornier-3_P5.08mm, symbol Device:R_POT
- added J3: POT3, TerminalBlock:TerminalBlock_bornier-3_P5.08mm, symbol Connector:Screw_Terminal_01x03
- added JP1: Pot3 Jumper, Jumper:SolderJumper-3_P1.3mm_Bridged12_Pad1.0x1.5mm_NumberLabels, symbol Jumper:Jumper_3_Bridged12
- added MH0, MH1, MH2, MH3: MountingHole, MountingHole:MountingHole_3.2mm_M3, symbol Mechanical:MountingHole
Connections:
- wire segments 40 -> 44
Changed lines of the file:
@@
 EESchema Schematic File Version 4
-EELAYER 30 0
+LIBS:desklamp-cache
+EELAYER 26 0
 EELAYER END
 $Descr A4 11693 8268
@@
 Signal
 $Comp
-L Device:R_POT RV3
-U 1 1 602F751B
-P 4950 2450
-F 0 "RV3" H 4880 2496 50  0000 R CNN
-F 1 "POT3" H 4880 2405 50  0000 R CNN
-F 2 "TerminalBlock:TerminalBlock_bornier-3_P5.08mm" H 4950 2450 50  0001 C CNN
-F 3 "~" H 4950 2450 50  0001 C CNN
-	1    4950 2450
-	1    0    0    -1
-$EndComp
-$Comp
 L Device:R_POT RV2
 U 1 1 602F75E6
@@
 Wire Wire Line
 	5350 1650 5850 1650
-Wire Wire Line
-	4950 2600 5550 2600
-Wire Wire Line
-	5550 2600 5550 1850
 Wire Wire Line
 	5550 1850 5850 1850
@@
 Wire Wire Line
 	4400 1800 4400 2250
-Wire Wire Line
-	4950 2300 4950 2250
-Wire Wire Line
-	4950 2250 4400 2250
 Connection ~ 4400 2250
 Wire Wire Line
@@
 	1    0    0    -1
 $EndComp
+$Comp
+L Jumper:Jumper_3_Bridged12 JP1
+U 1 1 60334B3A
+P 5450 2550
+F 0 "JP1" V 5404 2617 50  0000 L CNN
+F 1 "Pot3 Jumper" V 5495 2617 50  0000 L CNN
+F 2 "Jumper:SolderJumper-3_P1.3mm_Bridged12_Pad1.0x1.5mm_NumberLabels" H 5450 2550 50  0001 C CNN
+F 3 "~" H 5450 2550 50  0001 C CNN
+	1    5450 2550
+	0    1    1    0
+$EndComp
+$Comp
+L Connector:Screw_Terminal_01x03 J3
+U 1 1 60334D9B
+P 4900 2450
+F 0 "J3" H 5000 2400 50  0000 C CNN
+F 1 "POT3" H 5050 2500 50  0000 C CNN
+F 2 "TerminalBlock:TerminalBlock_bornier-3_P5.08mm" H 4900 2450 50  0001 C CNN
+F 3 "~" H 4900 2450 50  0001 C CNN
+	1    4900 2450
+	-1   0    0    1
+$EndComp
+Wire Wire Line
+	5100 2250 5100 2350
+Wire Wire Line
+	4400 2250 5100 2250
+Wire Wire Line
+	5300 2550 5100 2550
+Wire Wire Line
+	5450 2300 5550 2300
+Wire Wire Line
+	5550 2300 5550 1850
+Wire Wire Line
+	5450 2800 7350 2800
+Wire Wire Line
+	7350 2800 7350 1850
+Wire Wire Line
+	7350 1850 6950 1850
+$Comp
+L Mechanical:MountingHole MH0
+U 1 1 603373F3
+P 1650 4000
+F 0 "MH0" H 1750 4046 50  0000 L CNN
+F 1 "MountingHole" H 1750 3955 50  0000 L CNN
+F 2 "MountingHole:MountingHole_3.2mm_M3" H 1650 4000 50  0001 C CNN
+F 3 "~" H 1650 4000 50  0001 C CNN
+	1    1650 4000
+	1    0    0    -1
+$EndComp
+$Comp
+L Mechanical:MountingHole MH1
+U 1 1 6033746D
+P 1650 4250
+F 0 "MH1" H 1750 4296 50  0000 L CNN
+F 1 "MountingHole" H 1750 4205 50  0000 L CNN
+F 2 "MountingHole:MountingHole_3.2mm_M3" H 1650 4250 50  0001 C CNN
+F 3 "~" H 1650 4250 50  0001 C CNN
+	1    1650 4250
+	1    0    0    -1
+$EndComp
+$Comp
+L Mechanical:MountingHole MH2
+U 1 1 603374C5
+P 1650 4500
+F 0 "MH2" H 1750 4546 50  0000 L CNN
+F 1 "MountingHole" H 1750 4455 50  0000 L CNN
+F 2 "MountingHole:MountingHole_3.2mm_M3" H 1650 4500 50  0001 C CNN
+F 3 "~" H 1650 4500 50  0001 C CNN
+	1    1650 4500
+	1    0    0    -1
+$EndComp
+$Comp
+L Mechanical:MountingHole MH3
+U 1 1 60337515
+P 1650 4750
+F 0 "MH3" H 1750 4796 50  0000 L CNN
+F 1 "MountingHole" H 1750 4705 50  0000 L CNN
+F 2 "MountingHole:MountingHole_3.2mm_M3" H 1650 4750 50  0001 C CNN
+F 3 "~" H 1650 4750 50  0001 C CNN
+	1    1650 4750
+	1    0    0    -1
+$EndComp
